File: hardware/ps2usb.kicad_sch (KiCad schematic)
At the start: 22 parts, among them J1 DIN8, J2 USB1035, J3 DIN8, J4 DB9_Female_MountingHoles, U1 CH559L-less, U2 MAX232

Commit message: Internal version, replaced connectors with headers
Parts:
- removed J1: DIN8, ps2usb:DIN8, symbol Library:DIN8
- removed N1: Housing, ps2usb:Enclosure, symbol Mechanical:Housing
- removed RN1: R_Pack04, Resistor_SMD:R_Array_Convex_4x1206, symbol Device:R_Pack04
- added J5: EXTP1, Connector_PinHeader_2.54mm:PinHeader_2x06_P2.54mm_Vertical, symbol Connector_Generic:Conn_02x06_Odd_Even
- J2: value USB1035 -> USB; footprint ps2usb:USB1035 -> Connector_PinHeader_2.54mm:PinHeader_2x04_P2.54mm_Vertical
- J3: value DIN8 -> Keyboard; footprint ps2usb:DIN8 -> Connector_PinHeader_2.54mm:PinHeader_1x04_P2.54mm_Vertical
- J4: value DB9_Female_MountingHoles -> Mouse; footprint Connector_Dsub:DSUB-9_Female_Horizontal_P2.77x2.84mm_EdgePinOffset4.94mm_Housed_MountingHolesOffset7.48mm -> Connector_PinHeader_2.54mm:PinHeader_2x05_P2.54mm_Vertical
Connections:
- net +3.3V: now also J5.11 (Pin_11)
- net +5V: now also J5.2 (Pin_2)
- net GND: now also J5.1 (Pin_1), J5.12 (Pin_12)
- new net EXT1: J5.3 (Pin_3)
- new net EXT2: J5.4 (Pin_4)
- new net EXT3: J5.5 (Pin_5)
- new net EXT4: J5.6 (Pin_6)
- new net EXT5: J5.7 (Pin_7)
- new net EXT6: J5.8 (Pin_8)
- new net EXT7: J5.9 (Pin_9)
- new net EXT8: J5.10 (Pin_10)
Other:
- note removed: "MOUSE"
